File: PCB Rev 2/VolumetricDisplay.kicad_pcb (KiCad board)
At the start: 4 copper layers, 48.5 x 56 mm, 149 parts, among them J1 USB_C_Receptacle_USB2.0_16P, J2 Conn_ARM_SWD_TagConnect_TC2030, Q1 DMN32D2LDF, Q2 DMN32D2LDF, Q3 DMN32D2LDF, Q4 DMN32D2LDF, SW4 TS-1088-AR02016, SW5 TS-1088-AR02016, U2 NCP718xSN330, U3 RP2354B, U4 DRV8311S, U5 DRV5055A1xDBZxQ1, Y1 Abracon ABM8-272-T3

Commit message: Routing Progress
Route the USB differential pair, various lines. Create ground pore.
Routing:
- net LED5: track 0.00 -> 38.6 mm
- net LED6: track 0.00 -> 38.5 mm
- net LED7: track 0.00 -> 38.5 mm
- net LED4: track 0.00 -> 38.5 mm
- net LED2: track 0.00 -> 38.5 mm
- net LED1: track 0.00 -> 38.5 mm
- net LED0: track 0.12 -> 38.6 mm
- net LED3: track 0.00 -> 38.5 mm
- net LED14: track 0.00 -> 36.1 mm, vias 0 -> 2
- net LED13: track 0.00 -> 33.5 mm, vias 0 -> 2
- net LED15: track 0.00 -> 32.5 mm, vias 0 -> 2
- net LED12: track 0.00 -> 31.0 mm, vias 0 -> 2
- net Net-(U3-GPIO2): track 0.00 -> 26.3 mm
- net /MCU/QSPI_CS: track 0.00 -> 25.5 mm
- net Net-(U3-GPIO3): track 0.00 -> 24.5 mm
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- added copper zone on B.Cu, net GND

Commit message: Worked on stuff
Routing:
- net Net-(D13-K): track 0.00 -> 60.1 mm, vias 0 -> 8
- net Net-(D10-K): track 0.00 -> 54.9 mm, vias 0 -> 8
- net Net-(D15-K): track 0.00 -> 53.3 mm, vias 0 -> 8
- net Net-(D11-K): track 0.00 -> 52.6 mm, vias 0 -> 9
- net Net-(D14-K): track 0.00 -> 51.6 mm, vias 0 -> 8
- net Net-(D12-K): track 0.00 -> 50.5 mm, vias 0 -> 10
- net Net-(D16-K): track 2.36 -> 50.6 mm, vias 1 -> 8
- net Net-(D1-K): track 0.00 -> 44.7 mm, vias 0 -> 1
- net LED9: track 1.56 -> 39.8 mm, vias 1 -> 2
- net Net-(U3-GPIO0): track 0.00 -> 36.9 mm
- net Net-(U3-GPIO6): track 0.00 -> 34.9 mm, vias 0 -> 2
- net LED11: track 2.51 -> 36.6 mm, vias 1 -> 2
- net LED10: track 2.02 -> 34.4 mm, vias 1 -> 2
- net Net-(U3-GPIO1): track 0.00 -> 32.0 mm
- net Net-(U3-GPIO5): track 0.00 -> 31.9 mm, vias 0 -> 2
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- added copper zone on In1.Cu, net 3V3

Commit message: Today's routing
Routing:
- net 5V: track 41.7 -> 123.2 mm, vias 6 -> 7
- net Net-(U3-GPIO12): track 0.00 -> 33.2 mm, vias 0 -> 2
- net LED8: track 0.00 -> 31.9 mm
- net Net-(U3-GPIO41/ADC1): track 0.00 -> 31.3 mm, vias 0 -> 2
- net Net-(U3-GPIO11): track 0.00 -> 31.3 mm, vias 0 -> 2
- net +1V1: track 6.36 -> 37.3 mm, vias 0 -> 2
- net USB_DET: track 0.00 -> 26.6 mm
- net 3V3: track 24.3 -> 47.6 mm, vias 0 -> 7
- net nRST: track 2.47 -> 18.6 mm, vias 0 -> 2
- net SWDIO: track 0.00 -> 14.2 mm, vias 0 -> 2
- net LED2: track 38.5 -> 51.6 mm, vias 0 -> 2
- net Net-(U3-VREG_LX): track 0.00 -> 12.8 mm
- net LED6: track 38.5 -> 48.0 mm, vias 0 -> 1
- net LED3: track 38.5 -> 46.1 mm, vias 0 -> 2
- net PWM_A_L: track 0.00 -> 3.66 mm
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